Commit message: Updated bro_run with new programs

File: description/robot.urdf.xacro (robot description, xacro)
@@ -1,4 +1,14 @@
 <?xml version="1.0"?>
 <robot xmlns:xacro="http://www.ros.org/wiki/xacro"  name="robot">
-     <xacro:include filename="robot_core.xacro" />
+    <xacro:arg name="use_ros2_control" default="true"/>
+    <xacro:include filename="robot_core.xacro" />
+    <xacro:if value="$(arg use_ros2_control)">
+        <xacro:include filename="ros2_control.xacro" />
+    </xacro:if>
+    <xacro:unless value="$(arg use_ros2_control)">
+        <xacro:include filename="gazebo_control.xacro" />
+    </xacro:unless>
+    <xacro:include filename="lidar.xacro" />
+    <xacro:include filename="camera.xacro" />
+    <!-- <xacro:include filename="depth_camera.xacro" /> -->
 </robot>

File: description/robot_core.xacro (robot description, xacro)
@@ -13,4 +13,7 @@
      <material name="black">
         <color rgba="0 0 0 1"/>
+     </material>
+     <material name="red">
+        <color rgba="1.0 0.0 0.0 1.0"/>
      </material>
      <link name= "base_link">
@@ -36,7 +39,10 @@
         </collision>
         <xacro:inertial_box mass="0.5" x="0.3" y="0.3" z="0.15">
-            <orgin xyz="0.15 0 0.075" rpy="0 0 0"/>
+            <origin xyz="0.15 0 0.075" rpy="0 0 0"/>
         </xacro:inertial_box>
      </link>
+     <gazebo reference="chasis">
+        <material>Gazebo/white</material>
+     </gazebo>
      <!--LEFT WHEEL LINK-->
      <joint name="left_wheel_joint" type="continuous">
@@ -55,11 +61,14 @@
         <collision>
             <geometry>
-                <cylinder radius="0.05" length="0.04"/>
+                <sphere radius="0.05"/>
             </geometry>
         </collision>
         <xacro:inertial_cylinder mass="0.1" length="0.04" radius="0.05">
-            <orgin xyz="0 0 0" rpy="0 0 0"/>
+            <origin xyz="0 0 0" rpy="0 0 0"/>
         </xacro:inertial_cylinder>
      </link>
+     <gazebo reference="left_wheel">
+        <material>Gazebo/Blue</material>
+     </gazebo>
      <!--right WHEEL LINK-->
      <joint name="right_wheel_joint" type="continuous">
@@ -78,17 +87,20 @@
         <collision>
             <geometry>
-                <cylinder radius="0.05" length="0.04"/>
+                <sphere radius="0.05"/>
             </geometry>
         </collision>
          <xacro:inertial_cylinder mass="0.1" length="0.04" radius="0.05">
-            <orgin xyz="0 0 0" rpy="0 0 0"/>
+            <origin xyz="0 0 0" rpy="0 0 0"/>
         </xacro:inertial_cylinder>
      </link>
+     <gazebo reference="right_wheel">
+        <material>Gazebo/Blue</material>
+     </gazebo>
      <!--caster wheel link-->
      <joint name="caster_wheel_joint" type="fixed">
-        <parent link="chasis"/>
-        <child link="caster_wheel"/>
-        <origin xyz="0.24 0 0"/>
-     </joint>
+         <parent link="chasis"/>
+         <child link="caster_wheel"/>
+         <origin xyz="0.24 0 0"/>
+    </joint>
     <link name="caster_wheel">
         <visual>
@@ -104,6 +116,11 @@
         </collision>
         <xacro:inertial_sphere mass="0.1" radius="0.05">
-            <orgin xyz="0 0 0" rpy="0 0 0"/>
+            <origin xyz="0 0 0" rpy="0 0 0"/>
         </xacro:inertial_sphere>
     </link>
+    <gazebo reference="caster_wheel">
+        <material>Gazebo/Black</material>
+        <mu1 value="0.001"/>
+        <mu2 value="0.01"/>
+     </gazebo>
 </robot>
